File: ProgrammingBoard/Connectors.kicad_sch (KiCad schematic)
At the start: 4 parts, among them J1 X0511FVS-24AS-LPV01, J1 X0511WVS-24AS-LPV01, J2 X0511FVS-24AS-LPV01, J2 X0511WVS-24AS-LPV01

Commit message: Remove LED driver
Connections:
- net INT2 is gone; now on net GND: J2.21 (Pin_21), J2.22 (Pin_22)
- net LED_EN is gone; now on net LED0: J2.17 (Pin_17), J2.18 (Pin_18)
- net RX is gone; now on net GND: J2.5 (Pin_5), J2.6 (Pin_6)
- net TX is gone; now on net SCL: J2.3 (Pin_3), J2.4 (Pin_4)
- net VSENSE is gone; now on net SWDCLK: J2.11 (Pin_11), J2.12 (Pin_12)
- net BUTTON: now also J2.15 (Pin_15), J2.16 (Pin_16); no longer J2.23 (Pin_23), J2.24 (Pin_24)
- net GND: now also J2.23 (Pin_23), J2.24 (Pin_24)
- net INT1: now also J2.7 (Pin_7), J2.8 (Pin_8); no longer J2.23 (Pin_23), J2.24 (Pin_24)
- net LED0: no longer J2.7 (Pin_7), J2.8 (Pin_8)
- net LED1: now also J2.19 (Pin_19), J2.20 (Pin_20); no longer J2.10 (Pin_10), J2.9 (Pin_9)
- net LED2: now also J2.21 (Pin_21), J2.22 (Pin_22); no longer J2.19 (Pin_19), J2.20 (Pin_20)
- net LED3: now also J2.23 (Pin_23), J2.24 (Pin_24); no longer J2.21 (Pin_21), J2.22 (Pin_22)
- net RESET: now also J2.13 (Pin_13), J2.14 (Pin_14); no longer J2.1 (Pin_1), J2.2 (Pin_2)
- net SCL: no longer J2.13 (Pin_13), J2.14 (Pin_14)
- net SDA: now also J2.1 (Pin_1), J2.2 (Pin_2); no longer J2.15 (Pin_15), J2.16 (Pin_16)
- net SWDCLK: no longer J2.1 (Pin_1), J2.2 (Pin_2)
- net SWDIO: now also J2.10 (Pin_10), J2.9 (Pin_9); no longer J2.3 (Pin_3), J2.4 (Pin_4)
- net VCC: now also J2.1 (Pin_1), J2.2 (Pin_2), J2.3 (Pin_3), J2.4 (Pin_4)

Commit message: Change led matrix routing for sinking current through mcu, sourcing from battery
Connections:
- net BUTTON: now also J2.23 (Pin_23), J2.24 (Pin_24); no longer J2.15 (Pin_15), J2.16 (Pin_16)
- net COL0: now also J1.3 (Pin_3), J1.4 (Pin_4); no longer J1.7 (Pin_7), J1.8 (Pin_8)
- net COL1: now also J1.5 (Pin_5), J1.6 (Pin_6); no longer J1.10 (Pin_10), J1.9 (Pin_9)
- net COL10: now also J1.23 (Pin_23), J1.24 (Pin_24); no longer J1.5 (Pin_5), J1.6 (Pin_6)
- net COL2: now also J1.7 (Pin_7), J1.8 (Pin_8); no longer J1.11 (Pin_11), J1.12 (Pin_12)
- net COL3: now also J1.10 (Pin_10), J1.9 (Pin_9); no longer J1.13 (Pin_13), J1.14 (Pin_14)
- net COL4: now also J1.11 (Pin_11), J1.12 (Pin_12); no longer J1.15 (Pin_15), J1.16 (Pin_16)
- net COL5: now also J1.13 (Pin_13), J1.14 (Pin_14); no longer J1.17 (Pin_17), J1.18 (Pin_18)
- net COL6: now also J1.15 (Pin_15), J1.16 (Pin_16); no longer J1.19 (Pin_19), J1.20 (Pin_20)
- net COL7: now also J1.17 (Pin_17), J1.18 (Pin_18); no longer J1.21 (Pin_21), J1.22 (Pin_22)
- net COL8: now also J1.19 (Pin_19), J1.20 (Pin_20); no longer J1.23 (Pin_23), J1.24 (Pin_24)
- net COL9: now also J1.21 (Pin_21), J1.22 (Pin_22); no longer J1.3 (Pin_3), J1.4 (Pin_4)
- net GND: now also J1.23 (Pin_23), J1.24 (Pin_24); no longer J1.23 (Pin_23), J1.24 (Pin_24)
- net LED0: now also J2.15 (Pin_15), J2.16 (Pin_16); no longer J2.17 (Pin_17), J2.18 (Pin_18)
- net LED1: now also J2.17 (Pin_17), J2.18 (Pin_18); no longer J2.19 (Pin_19), J2.20 (Pin_20)
- net LED2: now also J2.19 (Pin_19), J2.20 (Pin_20); no longer J2.21 (Pin_21), J2.22 (Pin_22)
- net LED3: now also J2.21 (Pin_21), J2.22 (Pin_22); no longer J2.23 (Pin_23), J2.24 (Pin_24)
- net ROW0: now also J1.3 (Pin_3), J1.4 (Pin_4); no longer J1.3 (Pin_3), J1.4 (Pin_4)
- net ROW1: now also J1.5 (Pin_5), J1.6 (Pin_6); no longer J1.5 (Pin_5), J1.6 (Pin_6)
- net ROW2: now also J1.7 (Pin_7), J1.8 (Pin_8); no longer J1.7 (Pin_7), J1.8 (Pin_8)
- net ROW3: now also J1.10 (Pin_10), J1.9 (Pin_9); no longer J1.10 (Pin_10), J1.9 (Pin_9)
- net ROW4: now also J1.11 (Pin_11), J1.12 (Pin_12); no longer J1.11 (Pin_11), J1.12 (Pin_12)
- net ROW5: now also J1.13 (Pin_13), J1.14 (Pin_14); no longer J1.13 (Pin_13), J1.14 (Pin_14)
- net ROW6: now also J1.15 (Pin_15), J1.16 (Pin_16); no longer J1.15 (Pin_15), J1.16 (Pin_16)
- net ROW7: now also J1.17 (Pin_17), J1.18 (Pin_18); no longer J1.17 (Pin_17), J1.18 (Pin_18)
- net ROW8: now also J1.19 (Pin_19), J1.20 (Pin_20); no longer J1.19 (Pin_19), J1.20 (Pin_20)
- net ROW9: now also J1.21 (Pin_21), J1.22 (Pin_22); no longer J1.21 (Pin_21), J1.22 (Pin_22)
Other:
- title: (none) -> WordWatch - Programming Board
