File: ControllerBoard/ControllerBoard.kicad_pcb (KiCad board)
At the start: 4 copper layers, 34 x 13 mm, 41 parts, among them J1 X0511WVS-24AS-LPV01, J2 X0511WVS-24AS-LPV01, SW1 RESET, U2 LIS2DE12, U3 nRF52810-QFxx, Y1 32.768kHz, Y2 32MHz

Commit message: Update control board silkscreen
Other:
- board text added: "WordWatch Control Board v1.0 Nov-23 (c) eggsampler"
- board text removed: "WordWatch Control Board v1.0 Oct-23 (c) eggsampler"
Changed lines of the file:
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@@
     )
     (stroke (width 0.15) (type solid)) (fill none) (layer "Edge.Cuts"))
-  (gr_text "WordWatch\nControl Board\nv1.0 Oct-23\n(c) eggsampler" (at 141.85942 85.25) (layer "B.SilkS")
+  (gr_text "WordWatch\nControl Board\nv1.0 Nov-23\n(c) eggsampler" (at 141.85942 85.25) (layer "B.SilkS")
     (effects (font (size 0.75 0.75) (thickness 0.1)) (justify bottom mirror))
   )
